File: board/board.kicad_pcb (KiCad board)
At the start: 2 copper layers, 21 x 13 mm, 1 part

Commit message: initial
Parts:
- removed LOGO1: Logo_Open_Hardware_Small, Symbol:OSHW-Symbol_6.7x6mm_SilkScreen
- added C1: 100nF, Capacitor_SMD:C_0603_1608Metric, F.Cu at (86.5, 77.9)
- added C10: 22uF, Capacitor_SMD:C_0603_1608Metric, F.Cu at (98.0, 80.3)
- added C2: 1uF, Capacitor_SMD:C_0402_1005Metric, F.Cu at (93.0, 82.7)
- added C3: 2.2uF, Capacitor_SMD:C_1206_3216Metric, F.Cu at (95.9, 77.6)
- added D1: DSS110U, Diode_SMD:D_SOD-323F, F.Cu at (95.2, 79.8)
- added J1: 013_PoE_rectified, on_edge:on_edge_2x05_device, F.Cu at (77.0, 80.6)
- added J2: 003_power, on_edge:on_edge_2x05_host, F.Cu at (114.0, 80.5)
- added L1: 22uH, Inductor_SMD:L_Taiyo-Yuden_NR-30xx, F.Cu at (95.4, 82.5)
- added R1: 59k, Resistor_SMD:R_0402_1005Metric, F.Cu at (90.0, 82.7)
- added R2: 100k, Resistor_SMD:R_0402_1005Metric, F.Cu at (91.0, 82.7)
- added R3: 41.2R, Resistor_SMD:R_0402_1005Metric, F.Cu at (86.5, 80.3)
- added R4: 24.9k, Resistor_SMD:R_0402_1005Metric, F.Cu at (89.0, 82.7)
- added R5: 100k, Resistor_SMD:R_0402_1005Metric, F.Cu at (92.1, 82.7)
- added U1: MP8007, Package_DFN_QFN:QFN-28-1EP_4x5mm_P0.5mm_EP2.65x3.65mm_ThermalVias, F.Cu at (90.4, 79.0)
Routing:
- net /Controller/5V: track 0.00 -> 75.7 mm, vias 0 -> 3
- net GND: track 0.00 -> 50.2 mm
- net Net-(J1-Pad9): track 0.00 -> 32.2 mm
- net /Controller/PoE-: track 0.00 -> 18.7 mm
- net /Controller/GNDPWR: track 0.00 -> 16.9 mm
- net /Controller/SW: track 0.00 -> 5.82 mm
- net /Controller/VCC: track 0.00 -> 3.08 mm
- net /Controller/CLASS: track 0.00 -> 2.72 mm
- net /Controller/FB2: track 0.00 -> 2.68 mm
- net /Controller/DET: track 0.00 -> 1.18 mm
- net /Controller/ILIM: track 0.00 -> 1.16 mm
- added copper zone on F.Cu, net /Controller/GNDPWR
Other:
- board size 21 x 13 mm -> 37 x 13 mm
- rule pad_to_mask_clearance: 0 -> 0.04
- board text added: "osf.003"
- board text added: "osf.013"
- board text added: "osf.b052.v1.0"
